Commit message: Added gazebo simulation and project.launch file to launch everything

File: urdf/robot.urdf.xacro (robot description, xacro)
@@ -8,10 +8,11 @@
     <xacro:property name="box_width" value="0.5"/>
     <xacro:property name="box_height" value="0.25"/>
-    <xacro:property name="wheel_mass" value="0.5"/>
-    <xacro:property name="box_mass" value="5"/>
+    <xacro:property name="wheel_mass" value="0.3"/>
+    <xacro:property name="box_mass" value="4"/>
     <xacro:property name="kinect_length" value="0.1"/>
     <xacro:property name="kinect_width" value="0.2"/>
     <xacro:property name="kinect_height" value="0.12"/>
     <xacro:property name="kinect_mass" value="1"/>
+    <xacro:include filename="$(find project)/urdf/robot.gazebo"/>
     <material name="blue">
         <color rgba="0 0 0.8 0.75" />
@@ -38,6 +39,6 @@
         </collision>
         <inertial>   <!-- CHANGE HERE THE REAL MASS AND INTERIA VALUES OF OUR ROBOT-->
-            <mass value="0.5" />
-            <inertia ixx="0.13" ixy="0.0" ixz="0.0" iyy="0.21" iyz="0.0" izz="0.13" />
+            <mass value="${box_mass}" />
+            <inertia ixx="0.625" ixy="0.0" ixz="0.0" iyy="1" iyz="0.0" izz="0.625" />
         </inertial>
     </link>
@@ -58,5 +59,5 @@
             <inertial>  <!-- CHANGE WHEEL INTERIAL VALUES HERE -->
                 <mass value="${wheel_mass}"/>
-                <inertia ixx="0.0001" ixy="0.0" ixz="0.0" iyy="0.0001" iyz="0.0" izz="0.0001" />
+                <inertia ixx="0.0008" ixy="0.0" ixz="0.0" iyy="0.0008" iyz="0.0" izz="0.0015" />
             </inertial>
         </link>
@@ -66,10 +67,30 @@
             <origin xyz="${reflect_x*(box_length/2)-(reflect_x*(wheel_diam/2))} ${reflect_y*(wheel_len+(box_width/2))} -0.1" rpy="0 0 0"/>
             <axis xyz="0 1 0"/>
+            <limit effort="300.0" velocity="100.0"/>
         </joint>
+        <!--TRANSMISSION TO TELL GAZEBO WHAT TO DO WITH THIS JOINT (WHEELS)-->
+        <transmission name="${prefix_x}_${prefix_y}_wheel_trans">
+            <type>transmission_interface/SimpleTransmission</type>
+            <actuator name="${prefix_x}_${prefix_y}_wheel_motor">
+                <hardwareInterface>hardware_interface/VelocityJointInterface</hardwareInterface>
+                <mechanicalReduction>1</mechanicalReduction>
+            </actuator>
+            <joint name="${prefix_x}_${prefix_y}_wheel_joint">
+                <hardwareInterface>hardware_interface/VelocityJointInterface</hardwareInterface>
+            </joint>
+        </transmission>
+        <!-- SOME PHYSICAL PROPERTIES FOR THE WHEELS TO BE SIMULATED-->
+        <gazebo reference="${prefix_x}_${prefix_y}_wheel">
+            <mu1 value="10000.0"/>
+            <mu2 value="10000.0"/>
+            <kp value="10000000.0" />
+            <kd value="1.0" />
+            <material>Gazebo/Grey</material>
+        </gazebo>
     </xacro:macro>
-    <xacro:wheel prefix_x="front" prefix_y="right" reflect_x="1" reflect_y="1"/>
-    <xacro:wheel prefix_x="front" prefix_y="left" reflect_x="1" reflect_y="-1"/>
-    <xacro:wheel prefix_x="back" prefix_y="right" reflect_x="-1" reflect_y="1"/>
-    <xacro:wheel prefix_x="back" prefix_y="left" reflect_x="-1" reflect_y="-1"/>
+    <xacro:wheel prefix_x="front" prefix_y="right" reflect_x="1" reflect_y="-1"/>
+    <xacro:wheel prefix_x="front" prefix_y="left" reflect_x="1" reflect_y="1"/>
+    <xacro:wheel prefix_x="back" prefix_y="right" reflect_x="-1" reflect_y="-1"/>
+    <xacro:wheel prefix_x="back" prefix_y="left" reflect_x="-1" reflect_y="1"/>
     <link name="kinect">
         <visual>

Commit message: Added the kinect camera

File: urdf/robot.urdf.xacro (robot description, xacro)
@@ -93,4 +93,5 @@
     <xacro:wheel prefix_x="back" prefix_y="right" reflect_x="-1" reflect_y="-1"/>
     <xacro:wheel prefix_x="back" prefix_y="left" reflect_x="-1" reflect_y="1"/>
+    <!-- LINK AND JOINT FOR THE KINECT CAMERA-->
     <link name="kinect">
         <visual>
@@ -108,5 +109,5 @@
         <inertial>
             <mass value="${kinect_mass}"/>
-            <inertia ixx="0.000375" ixy="0" ixz="0" iyy="0.000375" iyz="0" izz="0.000375"/>
+            <inertia ixx="1e-6" ixy="0" ixz="0" iyy="1e-6" iyz="0" izz="1e-6"/>
         </inertial>
     </link>
@@ -116,3 +117,29 @@
         <origin xyz="${(box_length/2)-(kinect_length/2)} 0 ${(box_height/2)+(kinect_height/2)}"/>
     </joint>
+        <!-- kinect optical link for fixing the point cloud view-->
+    <link name="kinect_optical">
+        <collision>
+            <origin xyz="0 0 0" rpy="0 0 0"/>
+            <geometry>
+                <box size="0.15 0.30 0.15"/>
+            </geometry>
+        </collision>
+        <visual>
+            <origin rpy="0 0 0" xyz="0 0 0"/>
+            <geometry>
+                <box size="0.05 0.05 0.05"/>
+            </geometry>
+        </visual>
+        <inertial>
+            <mass value="1e-5" />
+            <origin xyz="0 0 0" rpy="0 0 0"/>
+            <inertia ixx="1e-6" ixy="0" ixz="0" iyy="1e-6" iyz="0" izz="1e-6" />
+        </inertial>
+    </link>
+    <joint name="kinect_optical_joint" type="fixed">
+        <axis xyz="0 1 0"/>
+        <origin xyz="0 0 0" rpy="-1.57 0 -1.57"/>
+        <parent link="kinect"/>
+        <child link="kinect_optical"/>
+    </joint>
 </robot>

Commit message: Added imu sensor

File: urdf/robot.urdf.xacro (robot description, xacro)
@@ -143,3 +143,27 @@
         <child link="kinect_optical"/>
     </joint>
+    <link name="imu_sensor">
+        <visual>
+            <origin xyz="0 0 0" rpy="0 0 0"/>
+            <geometry>
+                <box size="0.05 0.05 0.02"/>
+            </geometry>
+        </visual>
+        <collision>
+            <origin xyz="0 0 0" rpy="0 0 0"/>
+            <geometry>
+                <box size="0.05 0.05 0.02"/>
+            </geometry>
+        </collision>
+        <inertial>
+            <mass value="1e-5" />
+            <origin xyz="0 0 0" rpy="0 0 0"/>
+            <inertia ixx="1e-6" ixy="0" ixz="0" iyy="1e-6" iyz="0" izz="1e-6" />
+        </inertial>
+    </link>
+    <joint name="imu_sensor_joint" type="fixed">
+        <parent link="base_link"/>
+        <child link="imu_sensor"/>
+        <origin xyz="0 0 0" rpy="0 0 0"/>
+    </joint>
 </robot>

Commit message: added SLAM(gmapping), global localization (amcl) and navigation (move_base)

File: urdf/robot.urdf.xacro (robot description, xacro)
@@ -8,10 +8,10 @@
     <xacro:property name="box_width" value="0.5"/>
     <xacro:property name="box_height" value="0.25"/>
-    <xacro:property name="wheel_mass" value="0.3"/>
-    <xacro:property name="box_mass" value="4"/>
+    <xacro:property name="wheel_mass" value="0.2"/>
+    <xacro:property name="box_mass" value="1"/>
     <xacro:property name="kinect_length" value="0.1"/>
     <xacro:property name="kinect_width" value="0.2"/>
     <xacro:property name="kinect_height" value="0.12"/>
-    <xacro:property name="kinect_mass" value="1"/>
+    <xacro:property name="kinect_mass" value="0.2"/>
     <xacro:include filename="$(find project)/urdf/robot.gazebo"/>
     <material name="blue">
@@ -42,6 +42,50 @@
             <inertia ixx="0.625" ixy="0.0" ixz="0.0" iyy="1" iyz="0.0" izz="0.625" />
         </inertial>
+<!--        THE CASTER-->
+        <visual name="caster">
+            <origin xyz="-0.2 0 -0.15" rpy="0 0 0" />
+            <geometry>
+                <sphere radius="0.05" />
+            </geometry>
+            <material name="black" />
+        </visual>
+        <collision>
+            <origin xyz="-0.20 0 -0.125" rpy="0 0 0" />
+            <geometry>
+                <sphere radius="0.05" />
+            </geometry>
+        </collision>
+        <inertial>
+            <mass value="0.2" />
+            <inertia ixx="0.001" ixy="0.0" ixz="0.0" iyy="0.001" iyz="0.0" izz="0.001" />
+        </inertial>
     </link>
     <xacro:macro name="wheel" params="prefix_x prefix_y reflect_x reflect_y">
+<!--           WHEELS SHAFT-->
+<!--        <link name="${prefix_x}_${prefix_y}_shaft">-->
+<!--            <visual>-->
+<!--                <origin xyz="0 0 0" rpy="${pi/2} 0 0"/>-->
+<!--                <geometry>-->
+<!--                    <cylinder length="0.07" radius="0.007"/>-->
+<!--                </geometry>-->
+<!--            </visual>-->
+<!--            <collision>-->
+<!--                <origin rpy="${pi/2} 0 0" xyz="0 0 0"/>-->
+<!--                <geometry>-->
+<!--                    <cylinder length="0.07" radius="0.007"/>-->
+<!--                </geometry>-->
+<!--            </collision>-->
+<!--            <inertial>  &lt;!&ndash; CHANGE SHAFT INTERIAL VALUES HERE &ndash;&gt;-->
+<!--                <mass value="0.2"/>-->
+<!--                <inertia ixx="0.0008" ixy="0.0" ixz="0.0" iyy="0.0008" iyz="0.0" izz="0.0015" />-->
+<!--            </inertial>-->
+<!--        </link>-->
+<!--        <joint name="${prefix_x}_${prefix_y}_shaft_joint" type="continuous">-->
+<!--            <parent link="base_link"/>-->
+<!--            <child link="${prefix_x}_${prefix_y}_shaft"/>-->
+<!--            <origin xyz="${reflect_x*((box_length/2)+0.06)-(reflect_x*(wheel_diam/2))} ${reflect_y*(wheel_len+(box_width/2))} -0.12" rpy="0 0 0"/>-->
+<!--            <axis xyz="0 1 0"/>-->
+<!--            <limit effort="300.0" velocity="100.0"/>-->
+<!--        </joint>-->
         <link name="${prefix_x}_${prefix_y}_wheel">
             <visual>
@@ -65,10 +109,10 @@
             <parent link="base_link"/>
             <child link="${prefix_x}_${prefix_y}_wheel"/>
-            <origin xyz="${reflect_x*(box_length/2)-(reflect_x*(wheel_diam/2))} ${reflect_y*(wheel_len+(box_width/2))} -0.1" rpy="0 0 0"/>
+            <origin xyz="${reflect_x*((box_length/2)+0.0)-(reflect_x*(wheel_diam/2))} ${reflect_y*(wheel_len+(box_width/2))} -0.09" rpy="0 0 0"/>
             <axis xyz="0 1 0"/>
             <limit effort="300.0" velocity="100.0"/>
         </joint>
-        <!--TRANSMISSION TO TELL GAZEBO WHAT TO DO WITH THIS JOINT (WHEELS)-->
-        <transmission name="${prefix_x}_${prefix_y}_wheel_trans">
+        <!--TRANSMISSION TO TELL GAZEBO WHAT TO DO WITH THIS JOINT (SHAFTS)-->
+        <transmission name="${prefix_x}_${prefix_y}_shaft_trans">
             <type>transmission_interface/SimpleTransmission</type>
             <actuator name="${prefix_x}_${prefix_y}_wheel_motor">
@@ -82,7 +126,7 @@
         <!-- SOME PHYSICAL PROPERTIES FOR THE WHEELS TO BE SIMULATED-->
         <gazebo reference="${prefix_x}_${prefix_y}_wheel">
-            <mu1 value="10000.0"/>
-            <mu2 value="10000.0"/>
-            <kp value="10000000.0" />
+            <mu1 value="200.0"/>
+            <mu2 value="100.0"/>
+            <kp value="1000000.0" />
             <kd value="1.0" />
             <material>Gazebo/Grey</material>
@@ -91,6 +135,6 @@
     <xacro:wheel prefix_x="front" prefix_y="right" reflect_x="1" reflect_y="-1"/>
     <xacro:wheel prefix_x="front" prefix_y="left" reflect_x="1" reflect_y="1"/>
-    <xacro:wheel prefix_x="back" prefix_y="right" reflect_x="-1" reflect_y="-1"/>
-    <xacro:wheel prefix_x="back" prefix_y="left" reflect_x="-1" reflect_y="1"/>
+<!--    <xacro:wheel prefix_x="back" prefix_y="right" reflect_x="-1" reflect_y="-1"/>-->
+<!--    <xacro:wheel prefix_x="back" prefix_y="left" reflect_x="-1" reflect_y="1"/>-->
     <!-- LINK AND JOINT FOR THE KINECT CAMERA-->
     <link name="kinect">

Commit message: Final update

File: urdf/robot.urdf.xacro (robot description, xacro)
@@ -5,13 +5,13 @@
     <xacro:property name="wheel_diam" value="0.2" />
     <xacro:property name="pi" value="3.1415" />
-    <xacro:property name="box_length" value="0.5"/>
-    <xacro:property name="box_width" value="0.5"/>
+    <xacro:property name="box_length" value="0.50"/>
+    <xacro:property name="box_width" value="0.50"/>
     <xacro:property name="box_height" value="0.25"/>
     <xacro:property name="wheel_mass" value="0.2"/>
-    <xacro:property name="box_mass" value="1"/>
-    <xacro:property name="kinect_length" value="0.1"/>
+    <xacro:property name="box_mass" value="8"/>
+    <xacro:property name="kinect_length" value="0.08"/>
     <xacro:property name="kinect_width" value="0.2"/>
-    <xacro:property name="kinect_height" value="0.12"/>
-    <xacro:property name="kinect_mass" value="0.2"/>
+    <xacro:property name="kinect_height" value="0.1"/>
+    <xacro:property name="kinect_mass" value="0.01"/>
     <xacro:include filename="$(find project)/urdf/robot.gazebo"/>
     <material name="blue">
@@ -44,5 +44,5 @@
 <!--        THE CASTER-->
         <visual name="caster">
-            <origin xyz="-0.2 0 -0.15" rpy="0 0 0" />
+            <origin xyz="-0.20 0 -0.12" rpy="0 0 0" />
             <geometry>
                 <sphere radius="0.05" />
@@ -51,5 +51,5 @@
         </visual>
         <collision>
-            <origin xyz="-0.20 0 -0.125" rpy="0 0 0" />
+            <origin xyz="-0.2 0 -0.12" rpy="0 0 0" />
             <geometry>
                 <sphere radius="0.05" />
@@ -57,5 +57,5 @@
         </collision>
         <inertial>
-            <mass value="0.2" />
+            <mass value="0.25" />
             <inertia ixx="0.001" ixy="0.0" ixz="0.0" iyy="0.001" iyz="0.0" izz="0.001" />
         </inertial>
@@ -109,5 +109,5 @@
             <parent link="base_link"/>
             <child link="${prefix_x}_${prefix_y}_wheel"/>
-            <origin xyz="${reflect_x*((box_length/2)+0.0)-(reflect_x*(wheel_diam/2))} ${reflect_y*(wheel_len+(box_width/2))} -0.09" rpy="0 0 0"/>
+            <origin xyz="${reflect_x*((box_length/2)-0.0)-(reflect_x*(wheel_diam/2))} ${reflect_y*(((wheel_len))+(box_width/2))} -0.07" rpy="0 0 0"/>
             <axis xyz="0 1 0"/>
             <limit effort="300.0" velocity="100.0"/>

Commit message: Final update

File: urdf/robot.urdf.xacro (robot description, xacro)
@@ -62,30 +62,4 @@
     </link>
     <xacro:macro name="wheel" params="prefix_x prefix_y reflect_x reflect_y">
-<!--           WHEELS SHAFT-->
-<!--        <link name="${prefix_x}_${prefix_y}_shaft">-->
-<!--            <visual>-->
-<!--                <origin xyz="0 0 0" rpy="${pi/2} 0 0"/>-->
-<!--                <geometry>-->
-<!--                    <cylinder length="0.07" radius="0.007"/>-->
-<!--                </geometry>-->
-<!--            </visual>-->
-<!--            <collision>-->
-<!--                <origin rpy="${pi/2} 0 0" xyz="0 0 0"/>-->
-<!--                <geometry>-->
-<!--                    <cylinder length="0.07" radius="0.007"/>-->
-<!--                </geometry>-->
-<!--            </collision>-->
-<!--            <inertial>  &lt;!&ndash; CHANGE SHAFT INTERIAL VALUES HERE &ndash;&gt;-->
-<!--                <mass value="0.2"/>-->
-<!--                <inertia ixx="0.0008" ixy="0.0" ixz="0.0" iyy="0.0008" iyz="0.0" izz="0.0015" />-->
-<!--            </inertial>-->
-<!--        </link>-->
-<!--        <joint name="${prefix_x}_${prefix_y}_shaft_joint" type="continuous">-->
-<!--            <parent link="base_link"/>-->
-<!--            <child link="${prefix_x}_${prefix_y}_shaft"/>-->
-<!--            <origin xyz="${reflect_x*((box_length/2)+0.06)-(reflect_x*(wheel_diam/2))} ${reflect_y*(wheel_len+(box_width/2))} -0.12" rpy="0 0 0"/>-->
-<!--            <axis xyz="0 1 0"/>-->
-<!--            <limit effort="300.0" velocity="100.0"/>-->
-<!--        </joint>-->
         <link name="${prefix_x}_${prefix_y}_wheel">
             <visual>

Commit message: Final update

File: urdf/robot.urdf.xacro (robot description, xacro)
@@ -85,5 +85,5 @@
             <origin xyz="${reflect_x*((box_length/2)-0.0)-(reflect_x*(wheel_diam/2))} ${reflect_y*(((wheel_len))+(box_width/2))} -0.07" rpy="0 0 0"/>
             <axis xyz="0 1 0"/>
-            <limit effort="300.0" velocity="100.0"/>
+            <limit effort="1000.0" velocity="100.0"/>
         </joint>
         <!--TRANSMISSION TO TELL GAZEBO WHAT TO DO WITH THIS JOINT (SHAFTS)-->
@@ -109,6 +109,4 @@
     <xacro:wheel prefix_x="front" prefix_y="right" reflect_x="1" reflect_y="-1"/>
     <xacro:wheel prefix_x="front" prefix_y="left" reflect_x="1" reflect_y="1"/>
-<!--    <xacro:wheel prefix_x="back" prefix_y="right" reflect_x="-1" reflect_y="-1"/>-->
-<!--    <xacro:wheel prefix_x="back" prefix_y="left" reflect_x="-1" reflect_y="1"/>-->
     <!-- LINK AND JOINT FOR THE KINECT CAMERA-->
     <link name="kinect">
